File: Tp1/ampliBjt/ampliBjt.kicad_pcb (KiCad board)
At the start: 2 copper layers, 55 x 40 mm, 24 parts, among them J1 Screw_Terminal_01x03, Q1 BC548

Commit message: BJT terminado
Parts:
- R3: value 10K -> 15K
- R4: value R -> 330K
- R5: value R -> 100K
- R6: value R -> 12K
- R7: value R -> 3,9K
Changed lines of the file:
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@@
       (effects (font (size 1 1) (thickness 0.15)))
     )
-    (fp_text value 10K (at 5.08 0 180) (layer F.SilkS)
+    (fp_text value 15K (at 5.08 0 180) (layer F.SilkS)
       (effects (font (size 1 1) (thickness 0.15)))
     )
@@
       (effects (font (size 1 1) (thickness 0.15)))
     )
-    (fp_text value R (at 5.08 0) (layer F.SilkS)
+    (fp_text value 330K (at 5.08 0) (layer F.SilkS)
       (effects (font (size 1 1) (thickness 0.15)))
     )
@@
       (effects (font (size 1 1) (thickness 0.15)))
     )
-    (fp_text value R (at 5.08 0) (layer F.SilkS)
+    (fp_text value 100K (at 5.08 0) (layer F.SilkS)
       (effects (font (size 1 1) (thickness 0.15)))
     )
@@
       (effects (font (size 1 1) (thickness 0.15)))
     )
-    (fp_text value R (at 5.08 0) (layer F.SilkS)
+    (fp_text value 12K (at 5.08 0) (layer F.SilkS)
       (effects (font (size 1 1) (thickness 0.15)))
     )
@@
       (effects (font (size 1 1) (thickness 0.15)))
     )
-    (fp_text value R (at 5.08 0) (layer F.SilkS)
+    (fp_text value 3,9K (at 5.08 0) (layer F.SilkS)
       (effects (font (size 1 1) (thickness 0.15)))
     )
@@
       (xy -2.549664 1.91989) (xy -2.469928 1.911165) (xy -2.400256 1.919918)) (layer F.SilkS) (width 0.01))
   )
-  (gr_text "A: RESP\nC: EC" (at 147.32 88.9) (layer F.SilkS)
-    (effects (font (size 1.5 1.5) (thickness 0.3)))
+  (gr_text "A: RESP\nC: EC" (at 143.51 88.9) (layer F.SilkS)
+    (effects (font (size 1.5 1.5) (thickness 0.3)) (justify left))
   )
   (gr_text G (at 116.84 105.156) (layer F.SilkS)
