File: Tp1/ampliBjt/ampliBjt.sch (KiCad schematic (older format))
At the start: 14 parts

Commit message: Mosfet terminado, BJT faltan las resistencias
Parts:
- added TP1: Atenuador, Connector_PinHeader_2.54mm:PinHeader_1x01_P2.54mm_Vertical, symbol Connector:TestPoint
- added TP2: VB, Connector_PinHeader_2.54mm:PinHeader_1x01_P2.54mm_Vertical, symbol Connector:TestPoint
- added TP3: VL, Connector_PinHeader_2.54mm:PinHeader_1x01_P2.54mm_Vertical, symbol Connector:TestPoint
- added TP4: GND, Connector_PinHeader_2.54mm:PinHeader_1x01_P2.54mm_Vertical, symbol Connector:TestPoint
- C1: renamed from C?; value CP -> 10uF; footprint (none) -> Capacitor_THT:CP_Radial_D5.0mm_P2.00mm
- C2, C3: renamed from C?; value CP -> 100uF; footprint (none) -> Capacitor_THT:CP_Radial_D6.3mm_P2.50mm
- J1: renamed from J?; footprint (none) -> TerminalBlock_MetzConnect:TerminalBlock_MetzConnect_Type055_RT01503HDWU_1x03_P5.00mm_Horizontal
- JP1: renamed from JP?; footprint (none) -> Connector_PinHeader_2.54mm:PinHeader_1x02_P2.54mm_Vertical
- R1: renamed from R?; value R -> 560; footprint (none) -> Resistor_THT:R_Axial_DIN0207_L6.3mm_D2.5mm_P10.16mm_Horizontal
- R2: renamed from R?; value R -> 33; footprint (none) -> Resistor_THT:R_Axial_DIN0207_L6.3mm_D2.5mm_P10.16mm_Horizontal
- R3: renamed from R?; value R -> 10K; footprint (none) -> Resistor_THT:R_Axial_DIN0207_L6.3mm_D2.5mm_P10.16mm_Horizontal
- R4, R5, R6, R7: renamed from R?; footprint (none) -> Resistor_THT:R_Axial_DIN0207_L6.3mm_D2.5mm_P10.16mm_Horizontal
- R8: renamed from R?; value R -> 12K; footprint (none) -> Resistor_THT:R_Axial_DIN0207_L6.3mm_D2.5mm_P10.16mm_Horizontal
- gave numbers to parts that had none: 1
Connections:
- wire segments 27 -> 30

Commit message: BJT terminado
Parts:
- R3: value 10K -> 15K
- R4: value R -> 330K
- R5: value R -> 100K
- R6: value R -> 12K
- R7: value R -> 3,9K
Changed lines of the file:
@@
 P 6450 5050
 F 0 "R7" H 6520 5096 50  0000 L CNN
-F 1 "R" H 6520 5005 50  0000 L CNN
+F 1 "3,9K" H 6520 5005 50  0000 L CNN
 F 2 "Resistor_THT:R_Axial_DIN0207_L6.3mm_D2.5mm_P10.16mm_Horizontal" V 6380 5050 50  0001 C CNN
 F 3 "~" H 6450 5050 50  0001 C CNN
@@
 P 6450 3700
 F 0 "R6" H 6520 3746 50  0000 L CNN
-F 1 "R" H 6520 3655 50  0000 L CNN
+F 1 "12K" H 6520 3655 50  0000 L CNN
 F 2 "Resistor_THT:R_Axial_DIN0207_L6.3mm_D2.5mm_P10.16mm_Horizontal" V 6380 3700 50  0001 C CNN
 F 3 "~" H 6450 3700 50  0001 C CNN
@@
 P 5850 3700
 F 0 "R4" H 5920 3746 50  0000 L CNN
-F 1 "R" H 5920 3655 50  0000 L CNN
+F 1 "330K" H 5920 3655 50  0000 L CNN
 F 2 "Resistor_THT:R_Axial_DIN0207_L6.3mm_D2.5mm_P10.16mm_Horizontal" V 5780 3700 50  0001 C CNN
 F 3 "~" H 5850 3700 50  0001 C CNN
@@
 P 5850 5050
 F 0 "R5" H 5920 5096 50  0000 L CNN
-F 1 "R" H 5920 5005 50  0000 L CNN
+F 1 "100K" H 5920 5005 50  0000 L CNN
 F 2 "Resistor_THT:R_Axial_DIN0207_L6.3mm_D2.5mm_P10.16mm_Horizontal" V 5780 5050 50  0001 C CNN
 F 3 "~" H 5850 5050 50  0001 C CNN
@@
 P 4950 4350
 F 0 "R3" V 4743 4350 50  0000 C CNN
-F 1 "10K" V 4834 4350 50  0000 C CNN
+F 1 "15K" V 4834 4350 50  0000 C CNN
 F 2 "Resistor_THT:R_Axial_DIN0207_L6.3mm_D2.5mm_P10.16mm_Horizontal" V 4880 4350 50  0001 C CNN
 F 3 "~" H 4950 4350 50  0001 C CNN
